Commit message: make it move in gazebo

File: robot_module/urdf/include/robot_macros.xacro (robot description, xacro)
@@ -124,6 +124,6 @@
             <child link="${prefix}_wheel"/>
             <origin xyz="${pos_x_joint} ${reflect*pos_y_joint} ${pos_z_joint}" rpy="0 0 0"/>
-            <!-- <limit effort="100" velocity="100"/>
-            <joint_properties damping="0.0" friction="0.0"/> -->
+            <limit effort="100" velocity="100"/>
+            <joint_properties damping="0.0" friction="0.0"/>
         </joint>
         <!-- set wheel link param for gazebo -->
@@ -136,6 +136,6 @@
             <material>Gazebo/Black</material>
         </gazebo>
-        <!--  -->
-        <transmission name="${prefix}_trans">
+        <!-- set transmission system -->
+        <transmission name="${prefix}_wheel_trans">
             <type>transmission_interface/SimpleTransmission</type>
             <joint name="${prefix}_wheel_joint">
@@ -144,5 +144,5 @@
             <actuator name="${prefix}_motor">
                 <hardwareInterface>hardware_interface/EffortJointInterface</hardwareInterface>
-                <mechanicalReduction>10</mechanicalReduction>
+                <mechanicalReduction>1</mechanicalReduction>
             </actuator>
         </transmission>

File: robot_module/urdf/my_bot.xacro (robot description, xacro)
@@ -4,5 +4,4 @@
     <xacro:property name="robot_name" value="my_bot"/>
     <xacro:include filename="$(find ${package_name})/urdf/include/robot_macros.xacro"/>
-    <xacro:include filename="$(find ${package_name})/urdf/include/sensor_macros.xacro"/>
     <!-- set config -->
     <xacro:property name="chassis_yaml" value="$(find ${package_name})/config/chassis.yaml"/>
@@ -27,7 +26,15 @@
                         wheel_prop="${wheel_props}"/>
     <!-- Camera -->
-    <xacro:camera parent_prop="${chassis_props}"
-                  parent_link="chassis" />
+    <!-- <xacro:include filename="$(find ${package_name})/urdf/include/sensor_macros.xacro"/> -->
+    <!-- <xacro:camera parent_prop="${chassis_props}"
+                  parent_link="chassis" /> -->
     <!-- load argument for gazebo -->
-    <xacro:include filename="$(find robot_module)/urdf/my_bot.gazebo"/>
+    <!-- <xacro:include filename="$(find robot_module)/urdf/my_bot.gazebo"/> -->
+    <gazebo>
+        <plugin name="gazebo_ros_control" filename="libgazebo_ros_control.so">
+            <robotNamespace>/my_bot</robotNamespace>
+            <robotSimType>gazebo_ros_control/DefaultRobotHWSim</robotSimType>
+            <!-- <legacyModeNS>True</legacyModeNS> -->
+        </plugin>
+    </gazebo>
 </robot>
